File: pcb/katori.kicad_pcb (KiCad board)
At the start: 4 copper layers, 221.9 x 106.1 mm, 98 parts, among them J1 JST ACH, J2 Solder, SW1 EC_SW, SW10 EC_SW, SW11 EC_SW, SW12 EC_SW, SW13 EC_SW, SW14 EC_SW, SW15 EC_SW, SW16 EC_SW, SW17 EC_SW, SW18 EC_SW, SW19 EC_SW, SW2 EC_SW, SW20 EC_SW, SW21 EC_SW, SW22 EC_SW, SW23 EC_SW, SW24 EC_SW, SW25 EC_SW, SW26 EC_SW, SW27 EC_SW, SW28 EC_SW, SW29 EC_SW, SW3 EC_SW, SW30 EC_SW, SW31 POWER, SW4 EC_SW, SW5 EC_SW, SW6 EC_SW, SW7 EC_SW, SW8 EC_SW, SW9 EC_SW, U1 SeeeduinoXIAO_Hybrid, U2 74HC4051, U3 OPA357AIDBVR, U4 74HC4051

Commit message: revision 2 and readme updates
Parts:
- moved R5 5.30 mm to (124.5, 132.8)
- moved R12 4.69 mm to (203.2, 127.9)
- moved C4 1.77 mm to (199.9, 129.2), turned to 22 degrees
- moved SW13 0.75 mm to (103.1, 83.2)
- moved PH28 0.75 mm to (190.0, 137.2)
- moved C1 0.75 mm to (119.0, 121.5)
- moved SW3 0.75 mm to (110.2, 65.5)
- moved PH15 0.75 mm to (209.1, 121.1)
- moved BUMP7 0.75 mm to (146.1, 90.0)
- moved SW30 0.75 mm to (209.4, 134.5)
- moved R7 0.75 mm to (175.7, 115.4)
- moved PH22 0.75 mm to (242.1, 65.6)
- moved SW10 0.75 mm to (254.1, 69.6)
- moved BUMP3 0.75 mm to (53.7, 91.1)
- moved SW27 0.75 mm to (108.0, 134.5)
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Connections:
- SW27 pad 2: COL10 -> COL0
- SW30 pad 1: COL11 -> COL9
Routing:
- net COL10: track 34.5 -> 21.5 mm
- net COL11: track 35.6 -> 25.2 mm
- net COL9: track 120.0 -> 129.6 mm
- net COL0: track 129.4 -> 138.7 mm
- net +3V3: track 11.9 -> 12.6 mm
- net GND: vias 509 -> 517
Other:
- board text added: "katori rev2 grassfedreeve"
- board text removed: "katori rev1 grassfedreeve"
