File: pcb/key_matrix.kicad_sch (KiCad schematic)
At the start: 30 parts, among them SW1 EC_SW, SW10 EC_SW, SW11 EC_SW, SW12 EC_SW, SW13 EC_SW, SW14 EC_SW, SW16 EC_SW, SW2 EC_SW, SW27 EC_SW, SW28 EC_SW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

Commit message: revision 2 and readme updates
Connections:
- net COL0: now also SW27.2
- net COL10: no longer SW27.2
- net COL11: no longer SW3.1
- net COL9: now also SW3.1
Changed lines of the file:
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@@
-	)
-	(junction
-		(at 199.39 96.52)
-		(diameter 0)
-		(color 0 0 0 0)
 	)
 	(junction
@@
 	)
 	(junction
+		(at 267.97 58.42)
+		(diameter 0)
+		(color 0 0 0 0)
+	)
+	(junction
 		(at 119.38 48.26)
 		(diameter 0)
@@
 	)
 	(junction
-		(at 104.14 96.52)
-		(diameter 0)
-		(color 0 0 0 0)
-	)
-	(junction
 		(at 191.77 63.5)
 		(diameter 0)
@@
 	)
 	(junction
+		(at 35.56 58.42)
+		(diameter 0)
+		(color 0 0 0 0)
+	)
+	(junction
 		(at 58.42 58.42)
 		(diameter 0)
@@
 	(wire
 		(pts
-			(xy 104.14 104.14) (xy 127 104.14)
-		)
-		(stroke
-			(width 0)
-			(type default)
-		)
-	)
-	(wire
-		(pts
 			(xy 151.13 109.22) (xy 151.13 101.6)
 		)
@@
 	(wire
 		(pts
-			(xy 104.14 95.25) (xy 104.14 96.52)
-		)
-		(stroke
-			(width 0)
-			(type default)
-		)
-	)
-	(wire
-		(pts
 			(xy 161.29 104.14) (xy 161.29 113.03)
 		)
@@
 	(wire
 		(pts
-			(xy 199.39 104.14) (xy 176.53 104.14)
-		)
-		(stroke
-			(width 0)
-			(type default)
-		)
-	)
-	(wire
-		(pts
-			(xy 199.39 95.25) (xy 199.39 96.52)
+			(xy 176.53 93.98) (xy 176.53 104.14)
 		)
 		(stroke
@@
 	(wire
 		(pts
+			(xy 35.56 96.52) (xy 104.14 96.52)
+		)
+		(stroke
+			(width 0)
+			(type default)
+		)
+	)
+	(wire
+		(pts
+			(xy 267.97 96.52) (xy 267.97 58.42)
+		)
+		(stroke
+			(width 0)
+			(type default)
+		)
+	)
+	(wire
+		(pts
 			(xy 73.66 39.37) (xy 73.66 48.26)
 		)
@@
 	(wire
 		(pts
+			(xy 199.39 96.52) (xy 267.97 96.52)
+		)
+		(stroke
+			(width 0)
+			(type default)
+		)
+	)
+	(wire
+		(pts
 			(xy 184.15 67.31) (xy 161.29 67.31)
 		)
@@
 	(wire
 		(pts
+			(xy 191.77 101.6) (xy 191.77 109.22)
+		)
+		(stroke
+			(width 0)
+			(type default)
+		)
+	)
+	(wire
+		(pts
 			(xy 88.9 82.55) (xy 111.76 82.55)
 		)
@@
 	(wire
 		(pts
-			(xy 104.14 96.52) (xy 104.14 104.14)
+			(xy 127 92.71) (xy 127 104.14)
 		)
 		(stroke
@@
 	(wire
 		(pts
-			(xy 199.39 96.52) (xy 199.39 104.14)
-		)
-		(stroke
-			(width 0)
-			(type default)
-		)
-	)
-	(wire
-		(pts
 			(xy 81.28 31.75) (xy 81.28 39.37)
 		)
@@
 	(wire
 		(pts
-			(xy 191.77 109.22) (xy 191.77 101.6)
-		)
-		(stroke
-			(width 0)
-			(type default)
-		)
-	)
-	(wire
-		(pts
 			(xy 111.76 63.5) (xy 134.62 63.5)
 		)
@@
 		(pts
 			(xy 119.38 67.31) (xy 142.24 67.31)
+		)
+		(stroke
+			(width 0)
+			(type default)
+		)
+	)
+	(wire
+		(pts
+			(xy 35.56 58.42) (xy 35.56 96.52)
 		)
 		(stroke
@@
 	(global_label "COL11"
 		(shape input)
-		(at 199.39 95.25 90)
+		(at 176.53 93.98 90)
 		(fields_autoplaced yes)
 		(effects
@@
 		)
 		(property "Intersheetrefs" "${INTERSHEET_REFS}"
-			(at 199.39 88.0809 90)
+			(at 176.53 86.8109 90)
 			(effects
 				(font
@@
 	(global_label "COL10"
 		(shape input)
-		(at 104.14 95.25 90)
+		(at 127 92.71 90)
 		(fields_autoplaced yes)
 		(effects
@@
 		)
 		(property "Intersheetrefs" "${INTERSHEET_REFS}"
-			(at 104.14 88.0809 90)
+			(at 127 85.5409 90)
 			(effects
 				(font
